Commit message: Organize the files of robot_description

File: roomblock_description/robots/roomblock.urdf.xacro (robot description, xacro)
@@ -8,3 +8,26 @@
   <xacro:include filename="$(find roomblock_description)/urdf/roomba500.urdf.xacro"/>
   <create/>
+  <material name="Grey">
+    <color rgba="0.2 0.2 0.2 1.0"/>
+  </material>
+  <joint name="block_joint" type="fixed">
+    <origin xyz="0 0 0.061" rpy="0 0 0" />
+    <parent link="base_link"/>
+    <child link="block_link" />
+  </joint>
+  <link name="block_link">
+    <visual>
+      <origin xyz="0 0 0" rpy="0 0 0" />
+      <geometry>
+	<mesh filename="package://roomblock_description/meshes/block.dae"/>
+      </geometry>
+      <material name="Grey" />
+    </visual>
+  </link>
+  <joint name="laser_joint" type="fixed">
+    <origin xyz="0 0 0.1308" rpy="0 0 ${M_PI}" />
+    <parent link="block_link" />
+    <child link="laser" />
+  </joint>
+  <link name="laser"/>
 </robot>

File: roomblock_description/urdf/roomba500.urdf.xacro (robot description, xacro)
@@ -235,24 +235,4 @@
 	    </inertial>
 	  </link>
-	  <joint name="laser_joint" type="fixed">
-	    <origin xyz="0 0 0.075" rpy="0 0 ${M_PI}" />
-	    <parent link="base_link" />
-	    <child link="laser" />
-	  </joint>
-	  <link name="laser">
-	    <visual>
-	      <geometry>
-	        <box size="0.02 0.035 0.002" />
-	      </geometry>
-	      <material name="Green" />
-	    </visual>
-	    <inertial>
-	      <mass value="0.001" />
-	      <origin xyz="0 0 0" />
-	      <inertia ixx="0.0001" ixy="0.0" ixz="0.0"
-	        iyy="0.0001" iyz="0.0"
-	        izz="0.0001" />
-	    </inertial>
-	  </link>
 	  <!-- Simulation sensors -->
 	  <sim_create/>

Commit message: Add raspi camera module link

File: roomblock_description/robots/roomblock.urdf.xacro (robot description, xacro)
@@ -31,3 +31,9 @@
   </joint>
   <link name="laser"/>
+  <joint name="camera_joint" type="fixed">
+    <origin xyz="0 0 0.1" rpy="0 0 0" />
+    <parent link="block_link" />
+    <child link="raspicam" />
+  </joint>
+  <link name="raspicam"/>
 </robot>

File: roomblock_description/urdf/roomba500.urdf.xacro (robot description, xacro)
@@ -6,237 +6,237 @@
   <property name="base_y" value="0.33" />
   <property name="M_PI" value="3.1415926535897931" />
-	  <xacro:macro name="create">
-	    <material name="Green">
-	      <color rgba="0.0 0.8 0.0 1.0"/>
-	    </material>
-	  <!-- base_footprint is a fictitious link(frame) that is on the ground right below base_link origin, navigation stack depends on this frame -->
-	  <link name="base_footprint">
-	    <visual>
-	      <origin xyz="0 0 0" rpy="0 0 0" />
-	      <geometry>
-	        <box size="0.001 0.001 0.001" />
-	      </geometry>
-	      <material name="Green" />
-	    </visual>
-	    <collision>
-	      <origin xyz="0 0 0.017" rpy="0 0 0" />
-	      <geometry>
-	       <box size="0.001 0.001 0.001" />
-	      </geometry>
-	    </collision>
-	  </link>
-	  <link name="base_link">
-	    <inertial>
-	      <mass value="2" />
-	      <origin xyz="0 0 0.0" />
-	      <inertia ixx="0.01" ixy="0.0" ixz="0.0"
-	        iyy="0.01" iyz="0.0" izz="0.5" />
-	    </inertial>
-	    <visual>
-	      <origin xyz=" 0 0 0.0308" rpy="0 0 0" />
-	      <geometry>
-	        <mesh filename="package://create_description/meshes/create_body.dae"/>
-	      </geometry>
-	    </visual>
-	    <collision>
-	      <origin xyz="0.0 0.0 0.0308" rpy="0 0 0" />
-	      <geometry>
-	        <cylinder length="0.0611632" radius="0.016495"/>
-	      </geometry>
-	    </collision>
-	  </link>
-	  <link name="wall_sensor_link">
-	    <inertial>
-	      <mass value="0.01" />
-	      <origin xyz="0 0 0"/>
-	      <inertia ixx="0.001" ixy="0.0" ixz="0.0"
-	        iyy="0.001" iyz="0.0" izz="0.001" />
-	    </inertial>
-	  </link>
-	  <link name="left_cliff_sensor_link">
-	    <inertial>
-	      <mass value="0.01" />
-	      <origin xyz="0 0 0"/>
-	      <inertia ixx="0.001" ixy="0.0" ixz="0.0"
-	        iyy="0.001" iyz="0.0" izz="0.001" />
-	    </inertial>
-	  </link>
-	  <link name="right_cliff_sensor_link">
-	    <inertial>
-	      <mass value="0.01" />
-	      <origin xyz="0 0 0"/>
-	      <inertia ixx="0.001" ixy="0.0" ixz="0.0"
-	        iyy="0.001" iyz="0.0" izz="0.001" />
-	    </inertial>
-	  </link>
-	  <link name="leftfront_cliff_sensor_link">
-	    <inertial>
-	      <mass value="0.01" />
-	      <origin xyz="0 0 0"/>
-	      <inertia ixx="1.0" ixy="0.0" ixz="0.0"
-	        iyy="0.01" iyz="0.0" izz="0.01" />
-	    </inertial>
-	  </link>
-	  <link name="rightfront_cliff_sensor_link">
-	    <inertial>
-	      <mass value="0.01" />
-	      <origin xyz="0 0 0"/>
-	      <inertia ixx="0.001" ixy="0.0" ixz="0.0"
-	        iyy="0.001" iyz="0.0" izz="0.001" />
-	    </inertial>
-	  </link>
-	  <joint name="base_footprint_joint" type="fixed">
-	    <origin xyz="0 0 0.017" rpy="0 0 0" />
-	    <parent link="base_footprint"/>
-	    <child link="base_link" />
-	  </joint>
-	  <joint name="base_wall_sensor_joint" type="fixed">
-	    <origin xyz="0.09 -0.120 0.042" rpy="0 0 -1.0" />
-	    <parent link="base_link"/>
-	    <child link="wall_sensor_link" />
-	  </joint>
-	  <joint name="base_left_cliff_sensor_joint" type="fixed">
-	    <origin xyz="0.07 0.14 0.01" rpy="0 1.57079 0" />
-	    <parent link="base_link"/>
-	    <child link="left_cliff_sensor_link" />
-	  </joint>
-	  <joint name="base_right_cliff_sensor_joint" type="fixed">
-	    <origin xyz="0.07 -0.14 0.01" rpy="0 1.57079 0" />
-	    <parent link="base_link"/>
-	    <child link="right_cliff_sensor_link" />
-	  </joint>
-	  <joint name="base_leftfront_cliff_sensor_joint" type="fixed">
-	    <origin xyz="0.15 0.04 0.01" rpy="0 1.57079 0" />
-	    <parent link="base_link"/>
-	    <child link="leftfront_cliff_sensor_link" />
-	  </joint>
-	  <joint name="base_rightfront_cliff_sensor_joint" type="fixed">
-	    <origin xyz="0.15 -0.04 0.01" rpy="0 1.57079 0" />
-	    <parent link="base_link"/>
-	    <child link="rightfront_cliff_sensor_link" />
-	  </joint>
-	  <link name="left_wheel_link">
-	    <inertial>
-	      <origin xyz="0 0 0"/>
-	      <mass value="0.01" />
-	      <inertia ixx="0.001" ixy="0.0" ixz="0.0"
-	        iyy="0.001" iyz="0.0" izz="0.001" />
-	    </inertial>
-	    <visual>
-	      <origin xyz="0 0 0" rpy="0 1.5707 1.5707" />
-	      <geometry>
-	        <cylinder radius="0.033" length = "0.023"/>
-	      </geometry>
-	    </visual>
-	    <collision>
-	      <origin xyz="0 0 0" rpy="0 1.5707 1.5707" />
-	      <geometry>
-	        <cylinder radius="0.033" length = "0.023"/>
-	      </geometry>
-	    </collision>
-	  </link>
-	  <joint name="left_wheel_joint" type="continuous">
-	    <origin xyz="0 0.13 0.015" rpy="0 0 0"/>
-	    <parent link="base_link"/>
-	    <child link="left_wheel_link"/>
-	    <axis xyz="0 1 0"/>
-	  </joint>
-	  <link name="right_wheel_link">
-	    <inertial>
-	      <origin xyz="0 0 0"/>
-	      <mass value="0.01" />
-	      <inertia ixx="0.001" ixy="0.0" ixz="0.0"
-	        iyy="0.001" iyz="0.0" izz="0.001" />
-	    </inertial>
-	    <visual>
-	      <origin xyz="0 0 0" rpy="0 1.5707 1.5707" />
-	      <geometry>
-	        <cylinder radius="0.033" length = "0.023"/>
-	      </geometry>
-	    </visual>
-	    <collision>
-	      <origin xyz="0 0 0" rpy="0 1.5707 1.5707" />
-	      <geometry>
-	        <cylinder radius="0.033" length = "0.023"/>
-	      </geometry>
-	    </collision>
-	  </link>
-	  <joint name="right_wheel_joint" type="continuous">
-	    <origin xyz="0 -0.13 0.015" rpy="0 0 0"/>
-	    <parent link="base_link"/>
-	    <child link="right_wheel_link"/>
-	    <axis xyz="0 1 0"/>
-	  </joint>
-	  <link name="rear_wheel_link">
-	    <inertial>
-	      <origin xyz="0 0 0"/>
-	      <mass value="0.001" />
-	      <inertia ixx="0.0001" ixy="0.0" ixz="0.0"
-	        iyy="0.0001" iyz="0.0" izz="0.0001" />
-	    </inertial>
-	    <visual>
-	      <origin xyz="0 0 0" rpy="0 1.5707 1.5707"/>
-	      <geometry>
-	        <sphere radius="0.015" />
-	      </geometry>
-	    </visual>
-	    <collision>
-	      <origin xyz="0 0 0" rpy="0 1.5707 1.5707" />
-	      <geometry>
-	        <sphere radius="0.015" />
-	      </geometry>
-	    </collision>
-	  </link>
-	  <!-- fixed because there's no transmission -->
-	  <joint name="rear_castor_joint" type="fixed">
-	    <origin xyz="-0.13 0 0.0" rpy="0 0 0"/>
-	    <parent link="base_link"/>
-	    <child link="rear_wheel_link"/>
-	    <axis xyz="0 1 0"/>
-	  </joint>
-	  <link name="front_wheel_link">
-	    <inertial>
-	      <origin xyz="0 0 0" />
-	      <mass value="0.01" />
-	      <inertia ixx="0.001" ixy="0.0" ixz="0.0"
-	        iyy="0.001" iyz="0.0" izz="0.001" />
-	    </inertial>
-	    <visual>
-	      <origin xyz="0 0 0" rpy="0 1.5707 1.5707"/>
-	      <geometry>
-	        <sphere radius="0.018" />
-	      </geometry>
-	    </visual>
-	    <collision>
-	      <origin xyz="0 0 0" rpy="0 1.5707 1.5707" />
-	      <geometry>
-	        <sphere radius="0.018" />
-	      </geometry>
-	    </collision>
-	  </link>
-	  <!-- fixed because there's no transmission -->
-	  <joint name="front_castor_joint" type="fixed">
-	    <origin xyz="0.13 0 0.0" rpy="0 0 0"/>
-	    <parent link="base_link"/>
-	    <child link="front_wheel_link"/>
-	    <axis xyz="0 1 0"/>
-	  </joint>
-	  <joint name="gyro_joint" type="fixed">
-	    <axis xyz="0 1 0" />
-	    <origin xyz="0 0 0.04" rpy="0 0 0" />
-	    <parent link="base_link"/>
-	    <child link="gyro_link"/>
-	  </joint>
-	  <link name="gyro_link">
-	    <inertial>
-	      <mass value="0.001" />
-	      <origin xyz="0 0 0" rpy="0 0 0" />
-	      <inertia ixx="0.0001" ixy="0" ixz="0" iyy="0.000001" iyz="0" izz="0.0001" />
-	    </inertial>
-	  </link>
-	  <!-- Simulation sensors -->
-	  <sim_create/>
-	  <sim_create_wall_sensor/>
-	  <sim_create_cliff_sensors/>
+  <xacro:macro name="create">
+    <material name="Green">
+      <color rgba="0.0 0.8 0.0 1.0"/>
+    </material>
+    <!-- base_footprint is a fictitious link(frame) that is on the ground right below base_link origin, navigation stack depends on this frame -->
+    <link name="base_footprint">
+      <visual>
+	<origin xyz="0 0 0" rpy="0 0 0" />
+	<geometry>
+	  <box size="0.001 0.001 0.001" />
+	</geometry>
+	<material name="Green" />
+      </visual>
+      <collision>
+	<origin xyz="0 0 0.017" rpy="0 0 0" />
+	<geometry>
+	  <box size="0.001 0.001 0.001" />
+	</geometry>
+      </collision>
+    </link>
+    <link name="base_link">
+      <inertial>
+	<mass value="2" />
+	<origin xyz="0 0 0.0" />
+	<inertia ixx="0.01" ixy="0.0" ixz="0.0"
+	         iyy="0.01" iyz="0.0" izz="0.5" />
+      </inertial>
+      <visual>
+	<origin xyz=" 0 0 0.0308" rpy="0 0 0" />
+	<geometry>
+	  <mesh filename="package://create_description/meshes/create_body.dae"/>
+	</geometry>
+      </visual>
+      <collision>
+	<origin xyz="0.0 0.0 0.0308" rpy="0 0 0" />
+	<geometry>
+	  <cylinder length="0.0611632" radius="0.016495"/>
+	</geometry>
+      </collision>
+    </link>
+    <link name="wall_sensor_link">
+      <inertial>
+	<mass value="0.01" />
+	<origin xyz="0 0 0"/>
+	<inertia ixx="0.001" ixy="0.0" ixz="0.0"
+	         iyy="0.001" iyz="0.0" izz="0.001" />
+      </inertial>
+    </link>
+    <link name="left_cliff_sensor_link">
+      <inertial>
+	<mass value="0.01" />
+	<origin xyz="0 0 0"/>
+	<inertia ixx="0.001" ixy="0.0" ixz="0.0"
+	         iyy="0.001" iyz="0.0" izz="0.001" />
+      </inertial>
+    </link>
+    <link name="right_cliff_sensor_link">
+      <inertial>
+	<mass value="0.01" />
+	<origin xyz="0 0 0"/>
+	<inertia ixx="0.001" ixy="0.0" ixz="0.0"
+	         iyy="0.001" iyz="0.0" izz="0.001" />
+      </inertial>
+    </link>
+    <link name="leftfront_cliff_sensor_link">
+      <inertial>
+	<mass value="0.01" />
+	<origin xyz="0 0 0"/>
+	<inertia ixx="1.0" ixy="0.0" ixz="0.0"
+	         iyy="0.01" iyz="0.0" izz="0.01" />
+      </inertial>
+    </link>
+    <link name="rightfront_cliff_sensor_link">
+      <inertial>
+	<mass value="0.01" />
+	<origin xyz="0 0 0"/>
+	<inertia ixx="0.001" ixy="0.0" ixz="0.0"
+	         iyy="0.001" iyz="0.0" izz="0.001" />
+      </inertial>
+    </link>
+    <joint name="base_footprint_joint" type="fixed">
+      <origin xyz="0 0 0.017" rpy="0 0 0" />
+      <parent link="base_footprint"/>
+      <child link="base_link" />
+    </joint>
+    <joint name="base_wall_sensor_joint" type="fixed">
+      <origin xyz="0.09 -0.120 0.042" rpy="0 0 -1.0" />
+      <parent link="base_link"/>
+      <child link="wall_sensor_link" />
+    </joint>
+    <joint name="base_left_cliff_sensor_joint" type="fixed">
+      <origin xyz="0.07 0.14 0.01" rpy="0 1.57079 0" />
+      <parent link="base_link"/>
+      <child link="left_cliff_sensor_link" />
+    </joint>
+    <joint name="base_right_cliff_sensor_joint" type="fixed">
+      <origin xyz="0.07 -0.14 0.01" rpy="0 1.57079 0" />
+      <parent link="base_link"/>
+      <child link="right_cliff_sensor_link" />
+    </joint>
+    <joint name="base_leftfront_cliff_sensor_joint" type="fixed">
+      <origin xyz="0.15 0.04 0.01" rpy="0 1.57079 0" />
+      <parent link="base_link"/>
+      <child link="leftfront_cliff_sensor_link" />
+    </joint>
+    <joint name="base_rightfront_cliff_sensor_joint" type="fixed">
+      <origin xyz="0.15 -0.04 0.01" rpy="0 1.57079 0" />
+      <parent link="base_link"/>
+      <child link="rightfront_cliff_sensor_link" />
+    </joint>
+    <link name="left_wheel_link">
+      <inertial>
+	<origin xyz="0 0 0"/>
+	<mass value="0.01" />
+	<inertia ixx="0.001" ixy="0.0" ixz="0.0"
+	         iyy="0.001" iyz="0.0" izz="0.001" />
+      </inertial>
+      <visual>
+	<origin xyz="0 0 0" rpy="0 1.5707 1.5707" />
+	<geometry>
+	  <cylinder radius="0.033" length = "0.023"/>
+	</geometry>
+      </visual>
+      <collision>
+	<origin xyz="0 0 0" rpy="0 1.5707 1.5707" />
+	<geometry>
+	  <cylinder radius="0.033" length = "0.023"/>
+	</geometry>
+      </collision>
+    </link>
+    <joint name="left_wheel_joint" type="continuous">
+      <origin xyz="0 0.13 0.015" rpy="0 0 0"/>
+      <parent link="base_link"/>
+      <child link="left_wheel_link"/>
+      <axis xyz="0 1 0"/>
+    </joint>
+    <link name="right_wheel_link">
+      <inertial>
+	<origin xyz="0 0 0"/>
+	<mass value="0.01" />
+	<inertia ixx="0.001" ixy="0.0" ixz="0.0"
+	         iyy="0.001" iyz="0.0" izz="0.001" />
+      </inertial>
+      <visual>
+	<origin xyz="0 0 0" rpy="0 1.5707 1.5707" />
+	<geometry>
+	  <cylinder radius="0.033" length = "0.023"/>
+	</geometry>
+      </visual>
+      <collision>
+	<origin xyz="0 0 0" rpy="0 1.5707 1.5707" />
+	<geometry>
+	  <cylinder radius="0.033" length = "0.023"/>
+	</geometry>
+      </collision>
+    </link>
+    <joint name="right_wheel_joint" type="continuous">
+      <origin xyz="0 -0.13 0.015" rpy="0 0 0"/>
+      <parent link="base_link"/>
+      <child link="right_wheel_link"/>
+      <axis xyz="0 1 0"/>
+    </joint>
+    <link name="rear_wheel_link">
+      <inertial>
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
Commit message: Fix camera position

File: roomblock_description/robots/roomblock.urdf.xacro (robot description, xacro)
@@ -32,5 +32,5 @@
   <link name="laser"/>
   <joint name="camera_joint" type="fixed">
-    <origin xyz="0 0 0.1" rpy="0 0 0" />
+    <origin xyz="0.04 0 0.1" rpy="0 ${M_PI/2} 0" />
     <parent link="block_link" />
     <child link="raspicam" />
