Commit message: Fix RPLIDAR orientation

File: roomblock_description/urdf/roomba500.urdf.xacro (robot description, xacro)
@@ -235,5 +235,5 @@
 	  </link>
 	  <joint name="laser_joint" type="fixed">
-	    <origin xyz="0 0 0.075" rpy="0 0 0" />
+	    <origin xyz="0 0 0.075" rpy="0 0 ${PI}" />
 	    <parent link="base_link" />
 	    <child link="laser" />

Commit message: Change to run amcl

File: roomblock_description/urdf/roomba500.urdf.xacro (robot description, xacro)
@@ -5,4 +5,5 @@
   <property name="base_x" value="0.33" />
   <property name="base_y" value="0.33" />
+  <property name="M_PI" value="3.1415926535897931" />
 	  <xacro:macro name="create">
 	    <material name="Green">
@@ -235,5 +236,5 @@
 	  </link>
 	  <joint name="laser_joint" type="fixed">
-	    <origin xyz="0 0 0.075" rpy="0 0 0" />
+	    <origin xyz="0 0 0.075" rpy="0 0 ${M_PI}" />
 	    <parent link="base_link" />
 	    <child link="laser" />

Commit message: Change link name for IMU

File: roomblock_description/urdf/roomba500.urdf.xacro (robot description, xacro)
@@ -222,11 +222,10 @@
       <axis xyz="0 1 0"/>
     </joint>
-    <joint name="gyro_joint" type="fixed">
-      <axis xyz="0 1 0" />
-      <origin xyz="0 0 0.04" rpy="0 0 0" />
-      <parent link="base_link"/>
-      <child link="gyro_link"/>
-    </joint>
-    <link name="gyro_link">
+    <joint name="imu_joint" type="fixed">
+      <origin xyz="0 0 0.025" rpy="0 0 0" />
+      <parent link="block_link"/>
+      <child link="imu_link"/>
+    </joint>
+    <link name="imu_link">
       <inertial>
 	<mass value="0.001" />

Commit message: Change imu_link orientation
Now it match to the latest CAD design

File: roomblock_description/urdf/roomba500.urdf.xacro (robot description, xacro)
@@ -223,5 +223,5 @@
     </joint>
     <joint name="imu_joint" type="fixed">
-      <origin xyz="0 0 0.025" rpy="0 0 0" />
+      <origin xyz="0.03 0 0.025" rpy="0 ${M_PI} ${M_PI/2}" />
       <parent link="block_link"/>
       <child link="imu_link"/>

Commit message: Fix xacro related warnings

File: roomblock_description/urdf/roomba500.urdf.xacro (robot description, xacro)
@@ -3,7 +3,7 @@
   <!-- Macro for TurtleBot body. Including Gazebo extensions, but does not include Kinect -->
   <xacro:include filename="$(find create_description)/urdf/create_gazebo.urdf.xacro"/>
-  <property name="base_x" value="0.33" />
-  <property name="base_y" value="0.33" />
-  <property name="M_PI" value="3.1415926535897931" />
+  <xacro:property name="base_x" value="0.33" />
+  <xacro:property name="base_y" value="0.33" />
+  <xacro:property name="M_PI" value="3.1415926535897931" />
   <xacro:macro name="create">
     <material name="Green">
